Commit message: fixed package name errors

File: Task01/urdf/hola_bot.urdf (robot description, URDF)
Before this commit: robot hola_bot, 4 links, 3 joints
Links:
- link base_link: geometry collision cylinder length=0.005 radius=0.15; visual mesh filename=package://Task01/meshes/base_link.STL
- link front_wheel: geometry collision cylinder length=0.02 radius=.03; visual mesh filename=package://Task01/meshes/wheel.STL
- link left_wheel: geometry collision cylinder length=0.02 radius=.03; visual mesh filename=package://Task01/meshes/wheel.STL
- link right_wheel: geometry collision cylinder length=0.02 radius=.03; visual mesh filename=package://Task01/meshes/wheel.STL

File: Task02/urdf/hola_bot.urdf (robot description, URDF)
Before this commit: robot hola_bot, 4 links, 3 joints
Links:
- link base_link: geometry collision cylinder length=0.005 radius=0.15; visual mesh filename=package://Task02/meshes/base_link.obj
- link front_wheel: geometry collision cylinder length=0.02 radius=.03; visual mesh filename=package://Task02/meshes/wheel.STL
- link left_wheel: geometry collision cylinder length=0.02 radius=.03; visual mesh filename=package://Task02/meshes/wheel.STL
- link right_wheel: geometry collision cylinder length=0.02 radius=.03; visual mesh filename=package://Task02/meshes/wheel.STL
